File: v1.0/hardware/picoco2.kicad_pcb (KiCad board)
At the start: 2 copper layers, 54 x 102.9 mm, 37 parts, among them J1 Conn_01x03_Female, J2 Conn_01x03_Female, J3 Micro_SD_Card, Q1 Q_PMOS_GSD, Q2 Q_PMOS_GSD, Q3 Q_NMOS_GDS, SW1 SW_Push, SW2 SW_Push, U1 PicoW, U2 scd30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

Commit message: update
Parts:
- removed BT3: CR1220, picoco2:CR1220-2
- removed C3: 10uF, Capacitor_SMD:C_0603_1608Metric_Pad1.08x0.95mm_HandSolder
- removed R13: 10K, Resistor_THT:R_Axial_DIN0204_L3.6mm_D1.6mm_P7.62mm_Horizontal
- removed R14: 10K, Resistor_SMD:R_0603_1608Metric_Pad0.98x0.95mm_HandSolder
- removed U5: PCF8523T, Package_SO:SOIC-8_3.9x4.9mm_P1.27mm
- added BT2: CR1220, picoco2:CR1220-2, F.Cu at (15.8, 88.2)
- added C1: 10uF, Capacitor_SMD:C_0603_1608Metric_Pad1.08x0.95mm_HandSolder, F.Cu at (21.6, 93.2)
- added R6: 10K, Resistor_SMD:R_0603_1608Metric_Pad0.98x0.95mm_HandSolder, F.Cu at (15.7, 87.4)
- added R7: 1K, Resistor_SMD:R_0603_1608Metric_Pad0.98x0.95mm_HandSolder, F.Cu at (18.9, 88.1)
- added U3: ssd1306, picoco2:ssd1306_b, F.Cu at (23.2, 26.9)
- BZ1: footprint Buzzer_Beeper:MagneticBuzzer_Kobitone_254-EMB84Q-RO -> picoco2:CUI_CMT-4023S-SMT-TR
- Q1: value Q_PMOS_GSD -> Q_PMOS_GDS; footprint Package_TO_SOT_SMD:SOT-23 -> Package_TO_SOT_THT:TO-220-3_Vertical
- Q3: value Q_NMOS_GDS -> Q_PMOS_GSD
- R10: footprint Resistor_THT:R_Axial_DIN0204_L3.6mm_D1.6mm_P7.62mm_Horizontal -> Resistor_SMD:R_0603_1608Metric_Pad0.98x0.95mm_HandSolder
- R8: footprint Resistor_SMD:R_0603_1608Metric_Pad0.98x0.95mm_HandSolder -> Resistor_THT:R_Axial_DIN0204_L3.6mm_D1.6mm_P7.62mm_Horizontal
- R9: value 1K -> 10K; footprint Resistor_SMD:R_0603_1608Metric_Pad0.98x0.95mm_HandSolder -> Resistor_THT:R_Axial_DIN0204_L3.6mm_D1.6mm_P7.62mm_Horizontal
- U4: value ssd1306 -> PCF8523T; footprint picoco2:ssd1306_a -> Package_SO:SOIC-8_3.9x4.9mm_P1.27mm
- moved R8 84.9 mm to (8.50, 7.39), turned to -90 degrees
- moved R10 83.5 mm to (20.5, 99.2)
- moved R9 65.4 mm to (8.40, 25.2)
- moved U4 64.3 mm to (7.20, 89.2), turned to -90 degrees
- moved Q1 63.0 mm to (16.6, 26.4), turned to 180 degrees
- moved Y1 26.6 mm to (7.40, 82.8), turned to 90 degrees
- moved Q2 25.4 mm to (24.9, 82.3), turned to 90 degrees
- moved J3 6.63 mm to (33.4, 91.5)
- moved Q3 4.87 mm to (47.4, 87.6)
- moved D2 4.50 mm to (42.7, 93.6)
- moved R12 4.50 mm to (42.2, 91.0)
- moved R3 4.50 mm to (42.2, 86.5)
- moved R4 4.50 mm to (42.2, 88.7)
- moved J2 3.25 mm to (51.9, 82.6)
- moved BZ1 2.45 mm to (44.4, 82.1)
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Connections:
- C2 pad 1: Net-(C2-Pad1) -> +3V3
- Q1 pad 2: VSYS -> VBAT_AAA
- Q1 pad 3: VBAT_AAA -> VSYS
- R10 pad 1: +3V3 -> SCD30_EN
- R10 pad 2: BUT_A -> GND
- R11 pad 2: BUT_A -> BUT_B
- R12 pad 1: SCD30_EN -> +3V3
- R12 pad 2: GND -> BUT_B
- R8 pad 1: Net-(J2-Pad2) -> +3V3
- R8 pad 2: GND -> BUT_A
- R9 pad 1: Net-(C2-Pad1) -> +3V3
- R9 pad 2: +3V3 -> BUT_A
- U4 pad 1: GND -> Net-(U4-Pad1)
- U4 pad 2: +3V3 -> Net-(U4-Pad2)
- U4 pad 3: SCL -> Net-(BT2-Pad1)
- U4 pad 4: SDA -> GND
- Y1 pad 1: Net-(U5-Pad2) -> Net-(U4-Pad2)
- Y1 pad 4: Net-(U5-Pad1) -> Net-(U4-Pad1)

Commit message: update
Parts:
- added R13: 10K, Resistor_THT:R_Axial_DIN0204_L3.6mm_D1.6mm_P7.62mm_Horizontal, F.Cu at (29.8, 32.1)
- added R14: 10K, Resistor_SMD:R_0603_1608Metric_Pad0.98x0.95mm_HandSolder, F.Cu at (39.6, 84.9)
- added SW3: SW_Push, Button_Switch_THT:SW_Tactile_SPST_Angled_PTS645Vx31-2LFS, F.Cu at (50.7, 26.7)
- R10, R6: footprint Resistor_SMD:R_0603_1608Metric_Pad0.98x0.95mm_HandSolder -> Resistor_THT:R_Axial_DIN0204_L3.6mm_D1.6mm_P7.62mm_Horizontal
- R7: value 1K -> 10K; footprint Resistor_SMD:R_0603_1608Metric_Pad0.98x0.95mm_HandSolder -> Resistor_THT:R_Axial_DIN0204_L3.6mm_D1.6mm_P7.62mm_Horizontal
- R8: footprint Resistor_THT:R_Axial_DIN0204_L3.6mm_D1.6mm_P7.62mm_Horizontal -> Resistor_SMD:R_0603_1608Metric_Pad0.98x0.95mm_HandSolder
- R9: value 10K -> 1K; footprint Resistor_THT:R_Axial_DIN0204_L3.6mm_D1.6mm_P7.62mm_Horizontal -> Resistor_SMD:R_0603_1608Metric_Pad0.98x0.95mm_HandSolder
- moved R8 79.0 mm to (20.2, 85.5), turned to 0 degrees
- moved R10 66.7 mm to (19.7, 32.5), turned to 180 degrees
- moved R9 65.1 mm to (34.9, 84.7), turned to 180 degrees
- moved R6 59.5 mm to (1.19, 29.7)
- moved R7 58.0 mm to (1.59, 32.7)
- moved BZ1 41.0 mm to (3.80, 87.5)
- moved D2 40.3 mm to (2.40, 93.8)
- moved R12 39.8 mm to (2.40, 91.2)
- moved Y1 38.0 mm to (44.5, 91.0)
- moved U4 37.5 mm to (43.5, 98.7)
- moved Q2 18.3 mm to (23.9, 100.6)
- moved R3 18.1 mm to (24.3, 89.3), turned to -90 degrees
- moved R4 12.8 mm to (30.0, 84.9), turned to 0 degrees
- moved R2 11.0 mm to (44.0, 26.5), turned to 180 degrees
- moved C2 10.3 mm to (10.7, 85.8), turned to 0 degrees
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Connections:
- R10 pad 1: SCD30_EN -> +3V3
- R10 pad 2: GND -> BUT_A
- R11 pad 2: BUT_B -> BUT_A
- R12 pad 1: +3V3 -> SCD30_EN
- R12 pad 2: BUT_B -> GND
- R6 pad 1: Net-(J2-Pad2) -> +3V3
- R6 pad 2: GND -> BUT_A
- R7 pad 1: Net-(C1-Pad1) -> +3V3
- R7 pad 2: +3V3 -> BUT_A
- R8 pad 1: +3V3 -> Net-(J2-Pad2)
- R8 pad 2: BUT_A -> GND
- R9 pad 1: +3V3 -> Net-(C1-Pad1)
- R9 pad 2: BUT_A -> +3V3
- SW2 pad 1: BUT_B -> BUT_A
