File: v1.0/hardware/picoco2.kicad_sch (KiCad schematic)
At the start: 37 parts, among them J1 Conn_01x03_Female, J2 Conn_01x03_Female, J3 Micro_SD_Card, Q1 Q_PMOS_GSD, Q2 Q_PMOS_GSD, Q3 Q_NMOS_GDS, SW1 SW_Push, SW2 SW_Push, U1 PicoW, U2 scd30, U4 ssd1306, U5 PCF8523T, Y1 32KHz

Commit message: update
Parts:
- removed Q1: Q_PMOS_GSD, Package_TO_SOT_SMD:SOT-23, symbol Device:Q_PMOS_GSD
- removed Q3: Q_NMOS_GDS, Package_TO_SOT_SMD:SOT-23, symbol Device:Q_NMOS_GDS
- added Q1: Q_PMOS_GDS, Package_TO_SOT_THT:TO-220-3_Vertical, symbol Device:Q_PMOS_GDS
- added Q3: Q_PMOS_GSD, Package_TO_SOT_SMD:SOT-23, symbol Device:Q_PMOS_GSD
- BZ1: footprint Buzzer_Beeper:MagneticBuzzer_Kobitone_254-EMB84Q-RO -> picoco2:CUI_CMT-4023S-SMT-TR
- U3: renamed from U4; footprint picoco2:ssd1306_a -> picoco2:ssd1306_b
- renumbered BT3 to BT2, C2 to C1, C3 to C2, R12 to R10, R13 to R11, R14 to R12, R8 to R6, R9 to R7, R10 to R8, R11 to R9, U5 to U4
Connections:
- net GND: now also Q3.3 (D)
- net SCD30_EN: now also Q3.1 (G)
- net SCD30_GND: now also Q3.2 (S)
- net VBAT_AAA: now also Q1.2 (D)
- net VBUS: now also Q1.1 (G)
- net VSYS: now also Q1.3 (S)

Commit message: update
Parts:
- added R? (x2): 10K, Resistor_THT:R_Axial_DIN0204_L3.6mm_D1.6mm_P7.62mm_Horizontal, symbol Device:R
- added SW?: SW_Push, Button_Switch_THT:SW_Tactile_SPST_Angled_PTS645Vx31-2LFS, symbol Switch:SW_Push
Connections:
- net +3V3: now also R?.1, R?.1
- net BUT_A: now also R?.2, R?.2, SW?.1
- net GND: now also SW?.2
Changed lines of the file:
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@@
   (junction (at 134.62 156.21) (diameter 0) (color 0 0 0 0)
   )
+  (junction (at 148.59 92.71) (diameter 0) (color 0 0 0 0)
+  )
   (junction (at 134.62 148.59) (diameter 0) (color 0 0 0 0)
   )
@@
   (junction (at 93.98 48.26) (diameter 0) (color 0 0 0 0)
   )
+  (junction (at 148.59 100.33) (diameter 0) (color 0 0 0 0)
+  )
   (junction (at 134.62 162.56) (diameter 0) (color 0 0 0 0)
   )
@@
   (junction (at 93.98 30.48) (diameter 0) (color 0 0 0 0)
   )
+  (junction (at 148.59 106.68) (diameter 0) (color 0 0 0 0)
+  )
   (junction (at 39.37 43.18) (diameter 0) (color 0 0 0 0)
   )
@@
     (stroke (width 0) (type default) (color 0 0 0 0))
   )
+  (wire (pts (xy 139.7 100.33) (xy 148.59 100.33))
+    (stroke (width 0) (type default) (color 0 0 0 0))
+  )
   (wire (pts (xy 34.29 187.96) (xy 45.72 187.96))
     (stroke (width 0) (type default) (color 0 0 0 0))
@@
     (stroke (width 0) (type default) (color 0 0 0 0))
   )
+  (wire (pts (xy 139.7 92.71) (xy 148.59 92.71))
+    (stroke (width 0) (type default) (color 0 0 0 0))
+  )
   (wire (pts (xy 106.68 48.26) (xy 106.68 68.58))
     (stroke (width 0) (type default) (color 0 0 0 0))
@@
     (stroke (width 0) (type default) (color 0 0 0 0))
   )
+  (wire (pts (xy 148.59 100.33) (xy 148.59 106.68))
+    (stroke (width 0) (type default) (color 0 0 0 0))
+  )
   (wire (pts (xy 93.98 68.58) (xy 95.25 68.58))
     (stroke (width 0) (type default) (color 0 0 0 0))
@@
     (stroke (width 0) (type default) (color 0 0 0 0))
   )
+  (wire (pts (xy 148.59 106.68) (xy 153.67 106.68))
+    (stroke (width 0) (type default) (color 0 0 0 0))
+  )
   (wire (pts (xy 45.72 187.96) (xy 45.72 181.61))
     (stroke (width 0) (type default) (color 0 0 0 0))
@@
   )
   (wire (pts (xy 55.88 144.78) (xy 55.88 166.37))
+    (stroke (width 0) (type default) (color 0 0 0 0))
+  )
+  (wire (pts (xy 144.78 106.68) (xy 148.59 106.68))
     (stroke (width 0) (type default) (color 0 0 0 0))
   )
@@
     (effects (font (size 1.27 1.27)) (justify right))
     (property "Intersheet References" "${INTERSHEET_REFS}" (id 0) (at 193.6507 71.0406 0)
+      (effects (font (size 1.27 1.27)) (justify right) hide)
+    )
+  )
+  (global_label "BUT_A" (shape input) (at 144.78 106.68 180) (fields_autoplaced)
+    (effects (font (size 1.27 1.27)) (justify right))
+    (property "Intersheet References" "${INTERSHEET_REFS}" (id 0) (at 136.7426 106.6006 0)
       (effects (font (size 1.27 1.27)) (justify right) hide)
     )
@@
     )
     (property "Datasheet" "" (id 3) (at 25.4 119.38 0)
+      (effects (font (size 1.27 1.27)) hide)
+    )
+    (pin "1")
+  )
+  (symbol (lib_id "power:+3V3") (at 148.59 92.71 0) (unit 1)
+    (in_bom yes) (on_board yes) (fields_autoplaced)
+    (property "Reference" "#PWR?" (id 0) (at 148.59 96.52 0)
+      (effects (font (size 1.27 1.27)) hide)
+    )
+    (property "Value" "+3V3" (id 1) (at 148.59 87.63 0))
+    (property "Footprint" "" (id 2) (at 148.59 92.71 0)
+      (effects (font (size 1.27 1.27)) hide)
+    )
+    (property "Datasheet" "" (id 3) (at 148.59 92.71 0)
       (effects (font (size 1.27 1.27)) hide)
     )
@@
     (pin "2")
   )
+  (symbol (lib_id "Device:R") (at 139.7 96.52 0) (unit 1)
+    (in_bom yes) (on_board yes) (fields_autoplaced)
+    (property "Reference" "R?" (id 0) (at 142.24 95.2499 0)
+      (effects (font (size 1.27 1.27)) (justify left))
+    )
+    (property "Value" "10K" (id 1) (at 142.24 97.7899 0)
+      (effects (font (size 1.27 1.27)) (justify left))
+    )
+    (property "Footprint" "Resistor_THT:R_Axial_DIN0204_L3.6mm_D1.6mm_P7.62mm_Horizontal" (id 2) (at 137.922 96.52 90)
+      (effects (font (size 1.27 1.27)) hide)
+    )
+    (property "Datasheet" "~" (id 3) (at 139.7 96.52 0)
+      (effects (font (size 1.27 1.27)) hide)
+    )
+    (pin "1")
+    (pin "2")
+  )
   (symbol (lib_id "power:GND") (at 257.81 130.81 0) (unit 1)
     (in_bom yes) (on_board yes) (fields_autoplaced)
@@
     (pin "2")
   )
+  (symbol (lib_id "power:GND") (at 163.83 106.68 0) (unit 1)
+    (in_bom yes) (on_board yes) (fields_autoplaced)
+    (property "Reference" "#PWR?" (id 0) (at 163.83 113.03 0)
+      (effects (font (size 1.27 1.27)) hide)
+    )
+    (property "Value" "GND" (id 1) (at 163.83 111.76 0))
+    (property "Footprint" "" (id 2) (at 163.83 106.68 0)
+      (effects (font (size 1.27 1.27)) hide)
+    )
+    (property "Datasheet" "" (id 3) (at 163.83 106.68 0)
+      (effects (font (size 1.27 1.27)) hide)
+    )
+    (pin "1")
+  )
   (symbol (lib_id "Device:R") (at 125.73 152.4 0) (unit 1)
     (in_bom yes) (on_board yes) (fields_autoplaced)
@@
     )
     (property "Datasheet" "~" (id 3) (at 144.78 157.48 0)
+      (effects (font (size 1.27 1.27)) hide)
+    )
+    (pin "1")
+    (pin "2")
+  )
+  (symbol (lib_id "Device:R") (at 148.59 96.52 0) (unit 1)
+    (in_bom yes) (on_board yes) (fields_autoplaced)
+    (property "Reference" "R?" (id 0) (at 151.13 95.2499 0)
+      (effects (font (size 1.27 1.27)) (justify left))
+    )
+    (property "Value" "10K" (id 1) (at 151.13 97.7899 0)
+      (effects (font (size 1.27 1.27)) (justify left))
+    )
+    (property "Footprint" "Resistor_THT:R_Axial_DIN0204_L3.6mm_D1.6mm_P7.62mm_Horizontal" (id 2) (at 146.812 96.52 90)
+      (effects (font (size 1.27 1.27)) hide)
+    )
+    (property "Datasheet" "~" (id 3) (at 148.59 96.52 0)
+      (effects (font (size 1.27 1.27)) hide)
+    )
+    (pin "1")
+    (pin "2")
+  )
+  (symbol (lib_id "Switch:SW_Push") (at 158.75 106.68 0) (unit 1)
+    (in_bom yes) (on_board yes) (fields_autoplaced)
+    (property "Reference" "SW?" (id 0) (at 158.75 99.06 0))
+    (property "Value" "SW_Push" (id 1) (at 158.75 101.6 0))
+    (property "Footprint" "Button_Switch_THT:SW_Tactile_SPST_Angled_PTS645Vx31-2LFS" (id 2) (at 158.75 101.6 0)
+      (effects (font (size 1.27 1.27)) hide)
+    )
+    (property "Datasheet" "~" (id 3) (at 158.75 101.6 0)
       (effects (font (size 1.27 1.27)) hide)
     )
@@
       (reference "#PWR024") (unit 1) (value "GND") (footprint "")
     )
+    (path "/6a9cfd3d-0bc2-413c-98ce-689ba8d04199"
+      (reference "#PWR?") (unit 1) (value "+3V3") (footprint "")
+    )
+    (path "/9d08917f-daaf-4224-aa90-1a7010fa9f6b"
+      (reference "#PWR?") (unit 1) (value "GND") (footprint "")
+    )
     (path "/dea8c086-3176-4223-947b-b11dc0a0cc23"
       (reference "BT1") (unit 1) (value "Battery") (footprint "Battery:BatteryHolder_Keystone_2468_2xAAA")
@@
       (reference "R12") (unit 1) (value "10K") (footprint "Resistor_SMD:R_0603_1608Metric_Pad0.98x0.95mm_HandSolder")
     )
+    (path "/7e11dc5d-bf26-4382-ae67-9eb046a1cb85"
+      (reference "R?") (unit 1) (value "10K") (footprint "Resistor_THT:R_Axial_DIN0204_L3.6mm_D1.6mm_P7.62mm_Horizontal")
+    )
+    (path "/d4642166-c670-4bbd-a2fb-1b698b416015"
+      (reference "R?") (unit 1) (value "10K") (footprint "Resistor_THT:R_Axial_DIN0204_L3.6mm_D1.6mm_P7.62mm_Horizontal")
+    )
     (path "/d3fbd5d9-edde-42e2-941e-f1cb0af1d541"
       (reference "SW1") (unit 1) (value "SW_Push") (footprint "Button_Switch_THT:SW_Tactile_SPST_Angled_PTS645Vx31-2LFS")
@@
       (reference "SW2") (unit 1) (value "SW_Push") (footprint "Button_Switch_THT:SW_Tactile_SPST_Angled_PTS645Vx31-2LFS")
     )
+    (path "/d676812e-723d-4971-a919-3455584c6df4"
+      (reference "SW?") (unit 1) (value "SW_Push") (footprint "Button_Switch_THT:SW_Tactile_SPST_Angled_PTS645Vx31-2LFS")
+    )
     (path "/6fcbac42-cd34-406e-afc8-373c1f2ca8b6"
